Commit message: new urdf

File: cubot_urdf/cubot_shipped.urdf (robot description, URDF)
Before this commit: robot cubot_shipped, 54 links, 53 joints
Links:
- link m01_still: geometry collision cylinder length=0.04 radius=0.01; collision mesh filename=meshes/still.stl
Joints:
- joint servo01: limit effort=5.8 velocity=1.2 -> lower=-2.09439510 upper=2.09439510 effort=5.8 velocity=1.2; type continuous -> revolute
- joint servo02: limit effort=5.8 velocity=1.2 -> lower=-2.09439510 upper=2.09439510 effort=5.8 velocity=1.2; type continuous -> revolute
- joint servo03: limit effort=5.8 velocity=1.2 -> lower=-2.09439510 upper=2.09439510 effort=5.8 velocity=1.2; type continuous -> revolute
- joint servo04: limit effort=5.8 velocity=1.2 -> lower=-2.09439510 upper=2.09439510 effort=5.8 velocity=1.2; type continuous -> revolute
- joint servo05: limit effort=5.8 velocity=1.2 -> lower=-2.09439510 upper=2.09439510 effort=5.8 velocity=1.2; type continuous -> revolute
- joint servo06: limit effort=5.8 velocity=1.2 -> lower=-2.09439510 upper=2.09439510 effort=5.8 velocity=1.2; type continuous -> revolute
- joint servo07: limit effort=5.8 velocity=1.2 -> lower=-2.09439510 upper=2.09439510 effort=5.8 velocity=1.2; type continuous -> revolute
- joint servo08: limit effort=5.8 velocity=1.2 -> lower=-2.09439510 upper=2.09439510 effort=5.8 velocity=1.2; type continuous -> revolute
- joint servo09: limit effort=5.8 velocity=1.2 -> lower=-2.09439510 upper=2.09439510 effort=5.8 velocity=1.2; type continuous -> revolute
- joint servo10: limit effort=5.8 velocity=1.2 -> lower=-2.09439510 upper=2.09439510 effort=5.8 velocity=1.2; type continuous -> revolute
- joint servo11: limit effort=5.8 velocity=1.2 -> lower=-2.09439510 upper=2.09439510 effort=5.8 velocity=1.2; type continuous -> revolute
- joint servo12: limit effort=5.8 velocity=1.2 -> lower=-2.09439510 upper=2.09439510 effort=5.8 velocity=1.2; type continuous -> revolute
- joint servo13: limit effort=5.8 velocity=1.2 -> lower=-2.09439510 upper=2.09439510 effort=5.8 velocity=1.2; type continuous -> revolute
- joint servo14: limit effort=5.8 velocity=1.2 -> lower=-2.09439510 upper=2.09439510 effort=5.8 velocity=1.2; type continuous -> revolute
- joint servo15: limit effort=5.8 velocity=1.2 -> lower=-2.09439510 upper=2.09439510 effort=5.8 velocity=1.2; type continuous -> revolute
- joint servo16: limit effort=5.8 velocity=1.2 -> lower=-2.09439510 upper=2.09439510 effort=5.8 velocity=1.2; type continuous -> revolute
- joint servo17: limit effort=5.8 velocity=1.2 -> lower=-2.09439510 upper=2.09439510 effort=5.8 velocity=1.2; type continuous -> revolute
- joint servo18: limit effort=5.8 velocity=1.2 -> lower=-2.09439510 upper=2.09439510 effort=5.8 velocity=1.2; type continuous -> revolute
- joint servo19: limit effort=5.8 velocity=1.2 -> lower=-2.09439510 upper=2.09439510 effort=5.8 velocity=1.2; type continuous -> revolute
- joint servo20: limit effort=5.8 velocity=1.2 -> lower=-2.09439510 upper=2.09439510 effort=5.8 velocity=1.2; type continuous -> revolute
- joint servo21: limit effort=5.8 velocity=1.2 -> lower=-2.09439510 upper=2.09439510 effort=5.8 velocity=1.2; type continuous -> revolute
- joint servo22: limit effort=5.8 velocity=1.2 -> lower=-2.09439510 upper=2.09439510 effort=5.8 velocity=1.2; type continuous -> revolute
- joint servo23: limit effort=5.8 velocity=1.2 -> lower=-2.09439510 upper=2.09439510 effort=5.8 velocity=1.2; type continuous -> revolute
- joint servo24: limit effort=5.8 velocity=1.2 -> lower=-2.09439510 upper=2.09439510 effort=5.8 velocity=1.2; type continuous -> revolute
- joint servo25: limit effort=5.8 velocity=1.2 -> lower=-2.09439510 upper=2.09439510 effort=5.8 velocity=1.2; type continuous -> revolute
- joint servo26: limit effort=5.8 velocity=1.2 -> lower=-2.09439510 upper=2.09439510 effort=5.8 velocity=1.2; type continuous -> revolute
- joint servo27: limit effort=5.8 velocity=1.2 -> lower=-2.09439510 upper=2.09439510 effort=5.8 velocity=1.2; type continuous -> revolute
